Commit message: noi dung

File: install/open_manipulator_x_description/share/open_manipulator_x_description/gazebo/materials.xacro (robot description, xacro)
@@ -1,37 +1 @@
-<?xml version="1.0"?>
-<!--
-Copied from open_manipulator example -
-https://github.com/ROBOTIS-GIT/open_manipulator/blob/foxy-devel/open_manipulator_x_description/urdf/materials.xacro
--->
-<robot>
-  <material name="black">
-    <color rgba="0.0 0.0 0.0 1.0"/>
-  </material>
-  <material name="blue">
-    <color rgba="0.0 0.0 0.8 1.0"/>
-  </material>
-  <material name="brown">
-    <color rgba="0.8706 0.8118 0.7647 1.0"/>
-  </material>
-  <material name="dark">
-    <color rgba="0.3 0.3 0.3 1.0"/>
-  </material>
-  <material name="green">
-    <color rgba="0.0 0.8 0.0 1.0"/>
-  </material>
-  <material name="grey">
-    <color rgba="0.5 0.5 0.5 1.0"/>
-  </material>
-  <material name="light_black">
-    <color rgba="0.4 0.4 0.4 1.0"/>
-  </material>
-  <material name="orange">
-    <color rgba="1.0 0.4235 0.0392 1.0"/>
-  </material>
-  <material name="red">
-    <color rgba="0.8 0.0 0.0 1.0"/>
-  </material>
-  <material name="white">
-    <color rgba="1.0 1.0 1.0 1.0"/>
-  </material>
-</robot>
+/home/dung/Manipulator_amr_90_dergee/src/open_manipulator/open_manipulator_x_description/gazebo/materials.xacro

File: install/open_manipulator_x_description/share/open_manipulator_x_description/gazebo/open_manipulator_x.gazebo.xacro (robot description, xacro)
@@ -1,48 +1 @@
-<?xml version="1.0"?>
-<!--
-Copied and modified from turtlebot3 example:
-https://github.com/ROBOTIS-GIT/turtlebot3/blob/kinetic-devel/turtlebot3_description/urdf/turtlebot3_waffle_pi_for_open_manipulator.gazebo.xacro
--->
-<robot xmlns:xacro="http://ros.org/wiki/xacro">
-  <xacro:macro name="open_manipulator_x_gazebo" params="prefix">
-  <xacro:macro name="SimpleTransmission" params="trans joint actuator">
-    <transmission name="${trans}">
-      <type>transmission_interface/SimpleTransmission</type>
-      <joint name="${joint}">
-        <hardwareInterface>PositionJointInterface</hardwareInterface>
-      </joint>
-      <actuator name="${actuator}">
-        <mechanicalReduction>1</mechanicalReduction>
-        <hardwareInterface>PositionJointInterface</hardwareInterface>
-      </actuator>
-    </transmission>
-  </xacro:macro>
-  <xacro:macro name="Link" params="reference">
-    <gazebo reference="${reference}">
-      <kp>1000000.0</kp>
-      <kd>100.0</kd>
-      <mu1>30.0</mu1>
-      <mu2>30.0</mu2>
-      <maxVel>1.0</maxVel>
-      <minDepth>0.001</minDepth>
-      <material>Gazebo/DarkGrey</material>
-    </gazebo>
-  </xacro:macro>
-  <xacro:Link reference="${prefix}link1"/>
-  <xacro:Link reference="${prefix}link2"/>
-  <xacro:Link reference="${prefix}link3"/>
-  <xacro:Link reference="${prefix}link4"/>
-  <xacro:Link reference="${prefix}link5"/>
-  <xacro:Link reference="${prefix}gripper_left_link"/>
-  <xacro:Link reference="${prefix}gripper_right_link"/>
-  <gazebo reference="${prefix}end_effector_link">
-    <material>Gazebo/Red</material>
-  </gazebo>
-  <xacro:SimpleTransmission trans="${prefix}trans1" joint="${prefix}joint1" actuator="${prefix}actuator1" />
-  <xacro:SimpleTransmission trans="${prefix}trans2" joint="${prefix}joint2" actuator="${prefix}actuator2" />
-  <xacro:SimpleTransmission trans="${prefix}trans3" joint="${prefix}joint3" actuator="${prefix}actuator3" />
-  <xacro:SimpleTransmission trans="${prefix}trans4" joint="${prefix}joint4" actuator="${prefix}actuator4" />
-  <xacro:SimpleTransmission trans="${prefix}trans5" joint="${prefix}gripper_left_joint" actuator="${prefix}actuator5" />
-  <xacro:SimpleTransmission trans="${prefix}trans6" joint="${prefix}gripper_right_joint" actuator="${prefix}actuator6" />
-  </xacro:macro>
-</robot>
+/home/dung/Manipulator_amr_90_dergee/src/open_manipulator/open_manipulator_x_description/gazebo/open_manipulator_x.gazebo.xacro

File: install/open_manipulator_x_description/share/open_manipulator_x_description/ros2_control/open_manipulator_x_system.ros2_control.xacro (robot description, xacro)
@@ -1,177 +1 @@
-<?xml version="1.0"?>
-<robot xmlns:xacro="http://www.ros.org/wiki/xacro">
-  <xacro:macro name="open_manipulator_x_system" params="name prefix port_name:=/dev/ttyUSB0 use_sim:=^|false use_fake_hardware:=^|false fake_sensor_commands:=^|false">
-    <ros2_control name="${name}" type="system">
-      <xacro:if value="$(arg use_sim)">
-        <hardware>
-          <plugin>gazebo_ros2_control/GazeboSystem</plugin>
-        </hardware>
-      </xacro:if>
-      <xacro:unless value="$(arg use_sim)">
-        <hardware>
-          <xacro:if value="${use_fake_hardware}">
-            <plugin>fake_components/GenericSystem</plugin>
-            <param name="fake_sensor_commands">${fake_sensor_commands}</param>
-            <param name="state_following_offset">0.0</param>
-          </xacro:if>
-          <xacro:unless value="${use_fake_hardware}">
-            <plugin>dynamixel_hardware_interface/DynamixelHardware</plugin>
-            <param name="port_name">${port_name}</param>
-            <param name="baud_rate">1000000</param>
-            <param name="error_timeout_sec">0.2</param>
-            <param name="dynamixel_model_folder">/param/dxl_model</param>
-            <param name="number_of_joints">6</param>
-            <param name="number_of_transmissions">5</param>
-            <param name="transmission_to_joint_matrix">
-              1, 0, 0, 0, 0,
-              0, 1, 0, 0, 0,
-              0, 0, 1, 0, 0,
-              0, 0, 0, 1, 0,
-              0, 0, 0, 0, 1,
-              0, 0, 0, 0, 0
-            </param>
-            <param name="joint_to_transmission_matrix">
-              1, 0, 0, 0, 0, 0,
-              0, 1, 0, 0, 0, 0,
-              0, 0, 1, 0, 0, 0,
-              0, 0, 0, 1, 0, 0,
-              0, 0, 0, 0, 1, 0
-            </param>
-            <param name="ros_update_freq">200</param>
-            <param name="dynamixel_state_pub_msg_name">dynamixel_hardware_interface/dxl_state</param>
-            <param name="get_dynamixel_data_srv_name">dynamixel_hardware_interface/get_dxl_data</param>
-            <param name="set_dynamixel_data_srv_name">dynamixel_hardware_interface/set_dxl_data</param>
-            <param name="reboot_dxl_srv_name">dynamixel_hardware_interface/reboot_dxl</param>
-            <param name="set_dxl_torque_srv_name">dynamixel_hardware_interface/set_dxl_torque</param>
-              <!-- This parameter is used for a prismatic joint
-            that operates through a revolute mechanism. If the joint does not require this configuration, this parameter can be removed. -->
-            <param name="use_revolute_to_prismatic_gripper">1</param>
-            <param name="revolute_to_prismatic_dxl">dxl5</param>
-            <param name="revolute_max">-1.52</param>
-            <param name="revolute_min">0.92</param>
-            <param name="revolute_to_prismatic_joint">${prefix}gripper_left_joint</param>
-            <param name="prismatic_max">0.019</param>
-            <param name="prismatic_min">-0.01</param>
-          </xacro:unless>
-        </hardware>
-      </xacro:unless>
-      <joint name="${prefix}joint1">
-        <command_interface name="position"/>
-        <state_interface name="position"/>
-        <state_interface name="velocity"/>
-        <state_interface name="effort"/>
-      </joint>
-      <joint name="${prefix}joint2">
-        <command_interface name="position"/>
-        <state_interface name="position"/>
-        <state_interface name="velocity"/>
-        <state_interface name="effort"/>
-      </joint>
-      <joint name="${prefix}joint3">
-        <command_interface name="position"/>
-        <state_interface name="position"/>
-        <state_interface name="velocity"/>
-        <state_interface name="effort"/>
-      </joint>
-      <joint name="${prefix}joint4">
-        <command_interface name="position"/>
-        <state_interface name="position"/>
-        <state_interface name="velocity"/>
-        <state_interface name="effort"/>
-      </joint>
-      <joint name="${prefix}gripper_left_joint">
-        <command_interface name="position"/>
-        <state_interface name="position"/>
-        <state_interface name="velocity"/>
-        <state_interface name="effort"/>
-      </joint>
-      <joint name="${prefix}gripper_right_joint">
-        <param name="mimic">${prefix}gripper_left_joint</param>
-        <param name="multiplier">1</param>
-        <command_interface name="position"/>
-        <state_interface name="position"/>
-        <state_interface name="velocity"/>
-        <state_interface name="effort"/>
-      </joint>
-      <gpio name="dxl1">
-        <param name="type">dxl</param>
-        <param name="ID">11</param>
-        <command_interface name="Goal Position"/>
-        <state_interface name="Present Position"/>
-        <state_interface name="Present Velocity"/>
-        <state_interface name="Present Current"/>
-        <state_interface name="Torque Enable"/>
-        <state_interface name="Present Input Voltage"/>
-        <param name="Position P Gain">800</param>
-        <param name="Position I Gain">100</param>
-        <param name="Position D Gain">100</param>
-        <param name="Profile Velocity">200</param>
-        <param name="Profile Acceleration">50</param>
-        <param name="Drive Mode">0</param>
-        <param name="Return Delay Time">0</param>
-      </gpio>
-      <gpio name="dxl2">
-        <param name="type">dxl</param>
-        <param name="ID">12</param>
-        <command_interface name="Goal Position"/>
-        <state_interface name="Present Position"/>
-        <state_interface name="Present Velocity"/>
-        <state_interface name="Present Current"/>
-        <state_interface name="Torque Enable"/>
-        <state_interface name="Present Input Voltage"/>
-        <param name="Position P Gain">800</param>
-        <param name="Position I Gain">100</param>
-        <param name="Position D Gain">100</param>
-        <param name="Profile Velocity">200</param>
-        <param name="Profile Acceleration">50</param>
-        <param name="Drive Mode">0</param>
-        <param name="Return Delay Time">0</param>
-      </gpio>
-      <gpio name="dxl3">
-        <param name="type">dxl</param>
-        <param name="ID">13</param>
-        <command_interface name="Goal Position"/>
-        <state_interface name="Present Position"/>
-        <state_interface name="Present Velocity"/>
-        <state_interface name="Present Current"/>
-        <state_interface name="Torque Enable"/>
-        <state_interface name="Present Input Voltage"/>
-        <param name="Position P Gain">800</param>
-        <param name="Position I Gain">100</param>
-        <param name="Position D Gain">100</param>
-        <param name="Profile Velocity">200</param>
-        <param name="Profile Acceleration">50</param>
-        <param name="Drive Mode">0</param>
-        <param name="Return Delay Time">0</param>
-      </gpio>
-      <gpio name="dxl4">
-        <param name="type">dxl</param>
-        <param name="ID">14</param>
-        <command_interface name="Goal Position"/>
-        <state_interface name="Present Position"/>
-        <state_interface name="Present Velocity"/>
-        <state_interface name="Present Current"/>
-        <state_interface name="Torque Enable"/>
-        <state_interface name="Present Input Voltage"/>
-        <param name="Position P Gain">800</param>
-        <param name="Position I Gain">100</param>
-        <param name="Position D Gain">100</param>
-        <param name="Profile Velocity">200</param>
-        <param name="Profile Acceleration">50</param>
-        <param name="Drive Mode">0</param>
-        <param name="Return Delay Time">0</param>
-      </gpio>
-      <gpio name="dxl5">
-        <param name="type">dxl</param>
-        <param name="ID">15</param>
-        <command_interface name="Goal Position"/>
-        <state_interface name="Present Position"/>
-        <state_interface name="Present Velocity"/>
-        <state_interface name="Present Current"/>
-        <state_interface name="Torque Enable"/>
-        <state_interface name="Present Input Voltage"/>
-        <param name="Return Delay Time">0</param>
-      </gpio>
-    </ros2_control>
-  </xacro:macro>
-</robot>
+/home/dung/Manipulator_amr_90_dergee/src/open_manipulator/open_manipulator_x_description/ros2_control/open_manipulator_x_system.ros2_control.xacro

File: install/open_manipulator_x_description/share/open_manipulator_x_description/urdf/materials.xacro (robot description, xacro)
@@ -1,21 +1 @@
-<?xml version="1.0"?>
-<robot>
-  <material name="black">
-    <color rgba="0.0 0.0 0.0 1.0"/>
-  </material>
-  <material name="white">
-    <color rgba="1.0 1.0 1.0 1.0"/>
-  </material>
-  <material name="red">
-    <color rgba="0.8 0.0 0.0 1.0"/>
-  </material>
-  <material name="blue">
-    <color rgba="0.0 0.0 0.8 1.0"/>
-  </material>
-  <material name="green">
-    <color rgba="0.0 0.8 0.0 1.0"/>
-  </material>
-  <material name="grey">
-    <color rgba="0.5 0.5 0.5 1.0"/>
-  </material>
-</robot>
+/home/dung/Manipulator_amr_90_dergee/src/open_manipulator/open_manipulator_x_description/urdf/materials.xacro

File: install/open_manipulator_x_description/share/open_manipulator_x_description/urdf/open_manipulator_x.urdf.xacro (robot description, xacro)
@@ -1,230 +1 @@
-<?xml version="1.0"?>
-<robot xmlns:xacro="http://www.ros.org/wiki/xacro">
-  <xacro:macro name="open_manipulator_x" params="prefix=''">
-    <xacro:property
-      name="meshes_file_direction"
-      value="package://open_manipulator_x_description/meshes"/>
-    <link name="${prefix}link1">
-      <visual>
-        <origin xyz="0 0 0" rpy="0 0 0"/>
-        <geometry>
-          <mesh filename="${meshes_file_direction}/link1.stl" scale="0.001 0.001 0.001"/>
-        </geometry>
-        <material name="grey"/>
-      </visual>
-      <collision>
-        <origin xyz="0 0 0" rpy="0 0 0"/>
-        <geometry>
-          <mesh filename="${meshes_file_direction}/link1.stl" scale="0.001 0.001 0.001"/>
-        </geometry>
-      </collision>
-       <inertial>
-        <origin xyz="3.0876154e-04 0.0000000e+00 -1.2176461e-04" />
-        <mass value="7.9119962e-02" />
-        <inertia ixx="1.2505234e-05" ixy="0.0" ixz="-1.7855208e-07"
-                 iyy="2.1898364e-05" iyz="0.0"
-                 izz="1.9267361e-05" />
-      </inertial>
-    </link>
-    <joint name="${prefix}joint1" type="revolute">
-      <parent link="${prefix}link1"/>
-      <child link="${prefix}link2"/>
-      <origin xyz="0.012 0.0 0.017" rpy="0 0 0"/>
-      <axis xyz="0 0 1"/>
-      <limit velocity="4.8" effort="1" lower="${-pi}" upper="${pi}" />
-      <dynamics damping="0.1"/>
-    </joint>
-    <link name="${prefix}link2">
-      <visual>
-        <origin xyz="0 0 0.019" rpy="0 0 0"/>
-        <geometry>
-          <mesh filename="${meshes_file_direction}/link2.stl" scale="0.001 0.001 0.001"/>
-        </geometry>
-        <material name="grey"/>
-      </visual>
-      <collision>
-        <origin xyz="0 0 0.019" rpy="0 0 0"/>
-        <geometry>
-          <mesh filename="${meshes_file_direction}/link2.stl" scale="0.001 0.001 0.001"/>
-        </geometry>
-      </collision>
-       <inertial>
-        <origin xyz="-3.0184870e-04 5.4043684e-04 ${0.018 + 2.9433464e-02}" />
-        <mass value="9.8406837e-02" />
-        <inertia ixx="3.4543422e-05" ixy="-1.6031095e-08" ixz="-3.8375155e-07"
-                 iyy="3.2689329e-05" iyz="2.8511935e-08"
-                 izz="1.8850320e-05" />
-      </inertial>
-    </link>
-    <joint name="${prefix}joint2" type="revolute">
-      <parent link="${prefix}link2"/>
-      <child link="${prefix}link3"/>
-      <origin xyz="0.0 0.0 0.0595" rpy="0 0 0"/>
-      <axis xyz="0 1 0"/>
-      <limit velocity="4.8" effort="1" lower="${-1.5}" upper="${1.5}" />
-      <dynamics damping="0.1"/>
-    </joint>
-    <link name="${prefix}link3">
-      <visual>
-        <origin xyz="0 0 0" rpy="0 0 0"/>
-        <geometry>
-          <mesh filename="${meshes_file_direction}/link3.stl" scale="0.001 0.001 0.001"/>
-        </geometry>
-        <material name="grey"/>
-      </visual>
-      <collision>
-        <origin xyz="0 0 0" rpy="0 0 0"/>
-        <geometry>
-          <mesh filename="${meshes_file_direction}/link3.stl" scale="0.001 0.001 0.001"/>
-        </geometry>
-      </collision>
-       <inertial>
-        <origin xyz="1.0308393e-02 3.7743363e-04 1.0170197e-01" />
-        <mass value="1.3850917e-01" />
-        <inertia ixx="3.3055381e-04" ixy="-9.7940978e-08" ixz="-3.8505711e-05"
-                 iyy="3.4290447e-04" iyz="-1.5717516e-06"
-                 izz="6.0346498e-05" />
-      </inertial>
-    </link>
-    <joint name="${prefix}joint3" type="revolute">
-      <parent link="${prefix}link3"/>
-      <child link="${prefix}link4"/>
-      <origin xyz="0.024 0 0.128" rpy="0 0 0"/>
-      <axis xyz="0 1 0"/>
-      <limit velocity="4.8" effort="1" lower="${-1.5}" upper="${1.4}" />
-      <dynamics damping="0.1"/>
-    </joint>
-    <link name="${prefix}link4">
-      <visual>
-        <origin xyz="0 0 0" rpy="0 0 0"/>
-        <geometry>
-          <mesh filename="${meshes_file_direction}/link4.stl" scale="0.001 0.001 0.001"/>
-        </geometry>
-        <material name="grey"/>
-      </visual>
-      <collision>
-        <origin xyz="0 0 0" rpy="0 0 0"/>
-        <geometry>
-          <mesh filename="${meshes_file_direction}/link4.stl" scale="0.001 0.001 0.001"/>
-        </geometry>
-      </collision>
-       <inertial>
-        <origin xyz="9.0909590e-02 3.8929816e-04 2.2413279e-04" />
-        <mass value="1.3274562e-01" />
-        <inertia ixx="3.0654178e-05" ixy="-1.2764155e-06" ixz="-2.6874417e-07"
-                 iyy="2.4230292e-04" iyz="1.1559550e-08"
-                 izz="2.5155057e-04" />
-      </inertial>
-    </link>
-    <joint name="${prefix}joint4" type="revolute">
-      <parent link="${prefix}link4"/>
-      <child link="${prefix}link5"/>
-      <origin xyz="0.124 0.0 0.0" rpy="0 0 0"/>
-      <axis xyz="0 1 0"/>
-      <limit velocity="4.8" effort="1" lower="${-1.7}" upper="${1.97}" />
-      <dynamics damping="0.1"/>
-    </joint>
-    <link name="${prefix}link5">
-      <visual>
-        <origin xyz="0 0 0" rpy="0 0 0"/>
-        <geometry>
-          <mesh filename="${meshes_file_direction}/link5.stl" scale="0.001 0.001 0.001"/>
-        </geometry>
-        <material name="grey"/>
-      </visual>
-      <collision>
-        <origin xyz="0 0 0" rpy="0 0 0"/>
-        <geometry>
-          <mesh filename="${meshes_file_direction}/link5.stl" scale="0.001 0.001 0.001"/>
-        </geometry>
-      </collision>
-       <inertial>
-        <origin xyz="4.4206755e-02 3.6839985e-07 8.9142216e-03" />
-        <mass value="1.4327573e-01" />
-        <inertia ixx="8.0870749e-05" ixy="0.0" ixz="-1.0157896e-06"
-                 iyy="7.5980465e-05" iyz="0.0"
-                 izz="9.3127351e-05" />
-      </inertial>
-    </link>
-    <joint name="${prefix}gripper_left_joint" type="prismatic">
-      <parent link="${prefix}link5"/>
-      <child link="${prefix}gripper_left_link"/>
-      <origin xyz="0.0817 0.021 0.0" rpy="0 0 0"/>
-      <axis xyz="0 1 0"/>
-      <limit velocity="4.8" effort="1" lower="-0.010" upper="0.019" />
-      <dynamics damping="0.1"/>
-    </joint>
-    <link name="${prefix}gripper_left_link">
-      <visual>
-        <origin xyz="0 0 0" rpy="0 0 0"/>
-        <geometry>
-          <mesh filename="${meshes_file_direction}/gripper_left_palm.stl" scale="0.001 0.001 0.001"/>
-        </geometry>
-        <material name="grey"/>
-      </visual>
-      <collision>
-        <origin xyz="0 0 0" rpy="0 0 0"/>
-        <geometry>
-          <mesh filename="${meshes_file_direction}/gripper_left_palm.stl" scale="0.001 0.001 0.001"/>
-        </geometry>
-      </collision>
-      <inertial>
-        <origin xyz="0 0 0" />
-        <mass value="1.0e-03" />
-        <inertia ixx="1.0e-06" ixy="0.0" ixz="0.0"
-                 iyy="1.0e-06" iyz="0.0"
-                 izz="1.0e-06" />
-      </inertial>
-    </link>
-    <joint name="${prefix}gripper_right_joint_mimic" type="fixed">
-      <parent link="${prefix}gripper_right_link" />
-      <child link="dummy_mimic_fix" />
-    </joint>
-    <link name="dummy_mimic_fix"/>
-    <joint name="${prefix}gripper_right_joint" type="prismatic">
-      <parent link="${prefix}link5"/>
-      <child link="${prefix}gripper_right_link"/>
-      <origin xyz="0.0817 -0.021 0" rpy="0 0 0"/>
-      <axis xyz="0 -1 0"/>
-      <limit velocity="4.8" effort="1" lower="-0.010" upper="0.019" />
-      <mimic joint="${prefix}gripper_left_joint" multiplier="1"/>
-      <dynamics damping="0.1"/>
-    </joint>
-    <link name="${prefix}gripper_right_link">
-      <visual>
-        <origin xyz="0 0 0" rpy="0 0 0"/>
-        <geometry>
-          <mesh filename="${meshes_file_direction}/gripper_right_palm.stl" scale="0.001 0.001 0.001"/>
-        </geometry>
-        <material name="grey"/>
-      </visual>
-      <collision>
-        <origin xyz="0 0 0" rpy="0 0 0"/>
-        <geometry>
-          <mesh filename="${meshes_file_direction}/gripper_right_palm.stl" scale="0.001 0.001 0.001"/>
-        </geometry>
-      </collision>
-      <inertial>
-        <origin xyz="0 0 0" />
-        <mass value="1.0e-03" />
-        <inertia ixx="1.0e-06" ixy="0.0" ixz="0.0"
-                 iyy="1.0e-06" iyz="0.0"
-                 izz="1.0e-06" />
-      </inertial>
-    </link>
-    <joint name="${prefix}end_effector_joint" type="fixed">
-      <parent link="${prefix}link5"/>
-      <child link="${prefix}end_effector_link"/>
-      <origin xyz="0.126 0.0 0.0" rpy="0 0 0"/>
-    </joint>
-    <link name="${prefix}end_effector_link">
-      <visual>
-        <origin xyz="0 0 0" rpy="0 0 0"/>
-        <geometry>
-          <box size="0.01 0.01 0.01" />
-        </geometry>
-        <material name="red"/>
-       </visual>
-    </link>
-  </xacro:macro>
-</robot>
+/home/dung/Manipulator_amr_90_dergee/src/open_manipulator/open_manipulator_x_description/urdf/open_manipulator_x.urdf.xacro
