Commit message: noi dung

File: install/open_manipulator_x_description/share/open_manipulator_x_description/urdf/open_manipulator_x_robot.urdf.xacro (robot description, xacro)
@@ -1,36 +1 @@
-<?xml version="1.0"?>
-<!-- OpenManipulator Chain -->
-<robot name="open_manipulator_x" xmlns:xacro="http://ros.org/wiki/xacro">
-  <xacro:arg name="prefix" default="" />
-  <xacro:arg name="use_sim" default="false" />
-  <xacro:arg name="use_fake_hardware" default="false" />
-  <xacro:arg name="fake_sensor_commands" default="false" />
-  <xacro:arg name="port_name" default="/dev/ttyUSB0" />
-  <!-- Import Rviz colors -->
-  <xacro:include filename="$(find open_manipulator_x_description)/gazebo/materials.xacro" />
-  <!-- Import all Gazebo-customization elements, including Gazebo colors -->
-  <xacro:include filename="$(find open_manipulator_x_description)/gazebo/open_manipulator_x.gazebo.xacro" />
-  <!-- Import URDF -->
-  <xacro:include filename="$(find open_manipulator_x_description)/urdf/open_manipulator_x.urdf.xacro" />
-  <xacro:include filename="$(find open_manipulator_x_description)/ros2_control/open_manipulator_x_system.ros2_control.xacro" />
-  <xacro:open_manipulator_x prefix="$(arg prefix)" />
-  <xacro:open_manipulator_x_gazebo prefix="$(arg prefix)" />
-  <xacro:open_manipulator_x_system
-    name="OpenManipulatorXSystem" prefix="$(arg prefix)" use_sim="$(arg use_sim)"
-    use_fake_hardware="$(arg use_fake_hardware)"
-    fake_sensor_commands="$(arg fake_sensor_commands)"
-    port_name="$(arg port_name)"/>
-  <gazebo>
-    <plugin name="gazebo_ros2_control" filename="libgazebo_ros2_control.so">
-      <parameters>$(find open_manipulator_x_bringup)/config/gazebo_controller_manager.yaml</parameters>
-    </plugin>
-  </gazebo>
-  <!-- World -->
-  <link name="world"/>
-  <!-- World fixed joint-->
-  <joint name="$(arg prefix)world_fixed" type="fixed">
-    <origin xyz="0 0 0" rpy="0 0 0"/>
-    <parent link="world"/>
-    <child link="$(arg prefix)link1"/>
-  </joint>
-</robot>
+/home/dung/Manipulator_amr_90_dergee/src/open_manipulator/open_manipulator_x_description/urdf/open_manipulator_x_robot.urdf.xacro

File: install/open_manipulator_x_moveit_config/share/open_manipulator_x_moveit_config/config/open_manipulator_x.ros2_control.xacro (robot description, xacro)
@@ -1,47 +1 @@
-<?xml version="1.0"?>
-<robot xmlns:xacro="http://www.ros.org/wiki/xacro">
-    <xacro:macro name="open_manipulator_x_ros2_control" params="name initial_positions_file">
-        <xacro:property name="initial_positions" value="${load_yaml(initial_positions_file)['initial_positions']}"/>
-        <ros2_control name="${name}" type="system">
-            <hardware>
-                <!-- By default, set up controllers for simulation. This won't work on real hardware -->
-                <plugin>mock_components/GenericSystem</plugin>
-            </hardware>
-            <joint name="joint1">
-                <command_interface name="position"/>
-                <state_interface name="position">
-                  <param name="initial_value">${initial_positions['joint1']}</param>
-                </state_interface>
-                <state_interface name="velocity"/>
-            </joint>
-            <joint name="joint2">
-                <command_interface name="position"/>
-                <state_interface name="position">
-                  <param name="initial_value">${initial_positions['joint2']}</param>
-                </state_interface>
-                <state_interface name="velocity"/>
-            </joint>
-            <joint name="joint3">
-                <command_interface name="position"/>
-                <state_interface name="position">
-                  <param name="initial_value">${initial_positions['joint3']}</param>
-                </state_interface>
-                <state_interface name="velocity"/>
-            </joint>
-            <joint name="joint4">
-                <command_interface name="position"/>
-                <state_interface name="position">
-                  <param name="initial_value">${initial_positions['joint4']}</param>
-                </state_interface>
-                <state_interface name="velocity"/>
-            </joint>
-            <joint name="gripper_left_joint">
-                <command_interface name="position"/>
-                <state_interface name="position">
-                  <param name="initial_value">${initial_positions['gripper_left_joint']}</param>
-                </state_interface>
-                <state_interface name="velocity"/>
-            </joint>
-        </ros2_control>
-    </xacro:macro>
-</robot>
+/home/dung/Manipulator_amr_90_dergee/src/open_manipulator/open_manipulator_x_moveit_config/config/open_manipulator_x.ros2_control.xacro

File: install/open_manipulator_x_moveit_config/share/open_manipulator_x_moveit_config/config/open_manipulator_x.urdf.xacro (robot description, xacro)
@@ -1,9 +1 @@
-<?xml version="1.0"?>
-<robot xmlns:xacro="http://www.ros.org/wiki/xacro" name="open_manipulator_x">
-    <xacro:arg name="initial_positions_file" default="initial_positions.yaml" />
-    <!-- Import open_manipulator_x urdf file -->
-    <xacro:include filename="$(find open_manipulator_x_description)/urdf/open_manipulator_x_robot.urdf.xacro" />
-    <!-- Import control_xacro -->
-    <xacro:include filename="open_manipulator_x.ros2_control.xacro" />
-    <xacro:open_manipulator_x_ros2_control name="FakeSystem" initial_positions_file="$(arg initial_positions_file)"/>
-</robot>
+/home/dung/Manipulator_amr_90_dergee/src/open_manipulator/open_manipulator_x_moveit_config/config/open_manipulator_x.urdf.xacro

File: src/open_manipulator/open_manipulator_x_description/urdf/open_manipulator_x_robot.urdf.xacro (robot description, xacro)
@@ -21,4 +21,26 @@
     fake_sensor_commands="$(arg fake_sensor_commands)"
     port_name="$(arg port_name)"/>
+     <!-- ================= CAMERA ================= -->
+  <link name="camera_link">
+    <visual>
+      <geometry>
+        <box size="0.05 0.05 0.05"/>
+      </geometry>
+      <material name="blue"/>
+    </visual>
+  </link>
+  <!-- ✔ SỬA Ở ĐÂY -->
+  <joint name="camera_joint" type="fixed">
+    <parent link="$(arg prefix)world"/>
+    <child link="camera_link"/>
+    <origin xyz="-0.05 0 0.8" rpy="0 1.1869 0"/>
+  </joint>
+  <link name="camera_optical_frame"/>
+  <joint name="camera_optical_joint" type="fixed">
+    <parent link="camera_link"/>
+    <child link="camera_optical_frame"/>
+    <origin xyz="0 0 0" rpy="-1.5708 0 -1.5708"/>
+  </joint>
+  <!-- ================= END CAMERA ================= -->
   <gazebo>
     <plugin name="gazebo_ros2_control" filename="libgazebo_ros2_control.so">
@@ -30,5 +52,5 @@
   <!-- World fixed joint-->
   <joint name="$(arg prefix)world_fixed" type="fixed">
-    <origin xyz="0 0 0" rpy="0 0 0"/>
+    <origin xyz="0 0 0.02" rpy="0 0 0"/>
     <parent link="world"/>
     <child link="$(arg prefix)link1"/>
